Commit message: Rename mcav_sd_model to vehicle_model, add to README, suppress irrelevant warnings

File: visualisation/vehicle_model/urdf/bases/sd_twizy_body.urdf.xacro (robot description, xacro)
@@ -6,5 +6,5 @@
 -->
 <robot name="sd_twizy" xmlns:xacro="http://www.ros.org/wiki/xacro">
-  <xacro:include filename="$(find mcav_sd_model)/urdf/bases/sd_twizy_body.gazebo.xacro" />
+  <xacro:include filename="$(find vehicle_model)/urdf/bases/sd_twizy_body.gazebo.xacro" />
   <xacro:macro name="sd_twizy_base" params="name">
     <xacro:property name="depth" value="2.352"/>
@@ -39,5 +39,5 @@
         <origin xyz="0 0 0" rpy="0 0 1.57079632679"/>
         <geometry>
-          <mesh filename="file:///$(find mcav_sd_model)/meshes/SDTwizy.stl" scale="0.01 0.01 0.01"/>
+          <mesh filename="file:///$(find vehicle_model)/meshes/SDTwizy.stl" scale="0.01 0.01 0.01"/>
         </geometry>
         <material name="chassis_color" />
@@ -46,5 +46,5 @@
         <origin xyz="0 0 0" rpy="0 0 1.57079632679"/>
         <geometry>
-          <mesh filename="file:///$(find mcav_sd_model)/meshes/SDTwizy_collision.stl" scale="0.01 0.01 0.01"/>
+          <mesh filename="file:///$(find vehicle_model)/meshes/SDTwizy_collision.stl" scale="0.01 0.01 0.01"/>
         </geometry>
       </collision>

File: visualisation/vehicle_model/urdf/sd_twizy.urdf.xacro (robot description, xacro)
@@ -9,8 +9,8 @@
   <!-- Imported elements -->
   <!-- ***************** -->
-  <xacro:include filename="$(find mcav_sd_model)/urdf/bases/sd_twizy_body.urdf.xacro" />
-  <xacro:include filename="$(find mcav_sd_model)/urdf/wheels/sd_twizy_suspension.urdf.xacro" />
-  <xacro:include filename="$(find mcav_sd_model)/urdf/sensors/VLP-16.urdf.xacro"/>
-  <xacro:include filename="$(find mcav_sd_model)/urdf/sensors/cameras.urdf.xacro"/>
+  <xacro:include filename="$(find vehicle_model)/urdf/bases/sd_twizy_body.urdf.xacro" />
+  <xacro:include filename="$(find vehicle_model)/urdf/wheels/sd_twizy_suspension.urdf.xacro" />
+  <xacro:include filename="$(find vehicle_model)/urdf/sensors/VLP-16.urdf.xacro"/>
+  <xacro:include filename="$(find vehicle_model)/urdf/sensors/cameras.urdf.xacro"/>
   <!-- *************** -->
   <!-- Robots Elements -->

File: visualisation/vehicle_model/urdf/sensors/VLP-16.urdf.xacro (robot description, xacro)
@@ -18,10 +18,10 @@
             <visual>
                 <geometry>
-                    <mesh filename="file:///$(find mcav_sd_model)/meshes/VLP16_base_1.dae" />
+                    <mesh filename="file:///$(find vehicle_model)/meshes/VLP16_base_1.dae" />
                 </geometry>
             </visual>
             <visual>
                 <geometry>
-                    <mesh filename="file:///$(find mcav_sd_model)/meshes/VLP16_base_2.dae" />
+                    <mesh filename="file:///$(find vehicle_model)/meshes/VLP16_base_2.dae" />
                 </geometry>
             </visual>
@@ -47,5 +47,5 @@
                 <origin xyz="0 0 -0.0377" />
                 <geometry>
-                    <mesh filename="file:///$(find mcav_sd_model)/meshes/VLP16_scan.dae" />
+                    <mesh filename="file:///$(find vehicle_model)/meshes/VLP16_scan.dae" />
                 </geometry>
             </visual>
